Commit message: add two wheels on the robot

File: src/my_minimal_robot_description/urdf/minimal_robot.xacro (robot description, xacro)
@@ -2,6 +2,6 @@
 <robot name="minimal_robot" xmlns:xacro="http://ros.org/wiki/xacro">
   <!-- outer paramters（changing through launch file） -->
-  <xacro:arg name="base_height" default="0.5"/>
-  <xacro:arg name="sensor_size" default="0.2"/>
+  <xacro:arg name="base_height" default="0.2"/>
+  <xacro:arg name="sensor_size" default="0.1"/>
   <!-- inner paramters -->
   <xacro:property name="base_size" value="0.4"/>
@@ -9,4 +9,6 @@
   <xacro:property name="sensor_size"  value="$(arg sensor_size)"/>
   <xacro:property name="sensor_offset_z" value="${base_height/2 + sensor_size/2}"/>
+  <xacro:property name="wheel_radius" value="0.05"/>
+  <xacro:property name="wheel_width" value="0.02"/>
   <!-- base_link -->
   <link name="base_link">
@@ -39,3 +41,41 @@
     <axis xyz="0 0 1"/>
   </joint>
+  <!-- left wheel link -->
+  <link name="left_wheel_link">
+    <visual>
+      <origin xyz="0 0 0" rpy="1.5708 0 0"/>
+      <geometry>
+        <cylinder radius="${wheel_radius}" length="${wheel_width}"/>
+      </geometry>
+      <material name="black">
+        <color rgba="0 0 0 1.0"/>
+      </material>
+    </visual>
+  </link>
+  <!-- left wheel joint -->
+  <joint name="left_wheel_joint" type="continuous">
+    <parent link="base_link"/>
+    <child link="left_wheel_link"/>
+    <origin xyz="0 ${base_size/2} ${-base_height/2 + wheel_radius/2}" rpy="0 0 0"/>
+    <axis xyz="0 1 0"/>
+  </joint>
+  <!-- right wheel link -->
+  <link name="right_wheel_link">
+    <visual>
+      <origin xyz="0 0 0" rpy="1.5709 0 0"/>
+      <geometry>
+        <cylinder radius="${wheel_radius}" length="${wheel_width}"/>
+      </geometry>
+      <material name="black">
+        <color rgba="0 0 0 1.0"/>
+      </material>
+    </visual>
+  </link>
+  <!-- right wheel join -->
+  <joint name="right_wheel_joint" type="continuous">
+    <parent link="base_link"/>
+    <child link="right_wheel_link"/>
+    <origin xyz="0 ${-base_size/2} ${-base_height/2 + wheel_radius/2}" rpy="0 0 0"/>
+    <axis xyz="0 1 0"/>
+  </joint>
 </robot>

Commit message: learned diff drive robot and write xacro and launch file

File: src/my_minimal_robot_description/urdf/minimal_robot.xacro (robot description, xacro)
@@ -35,5 +35,5 @@
   </link>
   <!-- Joint：auto calculate the height of sensor -->
-  <joint name="base_to_sensor" type="continuous">
+  <joint name="base_to_sensor" type="fixed">
     <parent link="base_link"/>
     <child link="sensor_link"/>

Commit message: prepare for Gazebo

File: src/my_minimal_robot_description/urdf/minimal_robot.xacro (robot description, xacro)
@@ -9,6 +9,15 @@
   <xacro:property name="sensor_size"  value="$(arg sensor_size)"/>
   <xacro:property name="sensor_offset_z" value="${base_height/2 + sensor_size/2}"/>
-  <xacro:property name="wheel_radius" value="0.05"/>
-  <xacro:property name="wheel_width" value="0.02"/>
+  <xacro:property name="wheel_radius" value="0.1"/>
+  <xacro:property name="wheel_width" value="0.05"/>
+  <!-- base_footprint-->
+  <link name="base_footprint"/>
+  <joint name="base_footprint_to_base_link" type="fixed">
+  <parent link="base_footprint"/>
+  <child link="base_link"/>
+  <!-- 如果你希望 base_footprint 在 base_link 正下方某个高度，
+       可以在这里设置 xyz；目前简化成完全重合 -->
+  <origin xyz="0 0 0" rpy="0 0 0"/>
+  </joint>
   <!-- base_link -->
   <link name="base_link">
@@ -22,8 +31,22 @@
       </material>
     </visual>
+    <collision>
+        <origin xyz="0 0 0" rpy="0 0 0"/>
+        <geometry>
+          <box size="${base_size} ${base_size} ${base_height}"/>
+        </geometry>
+    </collision>
+    <inertial>
+        <mass value="1.0"/> <!-- kg -->
+        <inertia
+          ixx="0.01" ixy="0.0" ixz="0.0"
+          iyy="0.01" iyz="0.0"
+          izz="0.02"/>
+    </inertial>
   </link>
   <!-- sensor_link -->
   <link name="sensor_link">
     <visual>
+      <origin xyz="0 0 0" rpy="0 0 0"/>
       <geometry>
         <box size="${sensor_size} ${sensor_size} ${sensor_size}"/>
@@ -33,4 +56,17 @@
       </material>
     </visual>
+    <collision>
+      <origin xyz="0 0 0" rpy="0 0 0"/>
+      <geometry>
+        <box size="${sensor_size} ${sensor_size} ${sensor_size}"/>
+      </geometry>
+    </collision>
+    <inertial>
+      <mass value="0.05"/>
+      <inertia
+        ixx="0.00005" ixy="0.0" ixz="0.0"
+        iyy="0.00005" iyz="0.0"
+        izz="0.00005"/>
+    </inertial>
   </link>
   <!-- Joint：auto calculate the height of sensor -->
@@ -52,4 +88,17 @@
       </material>
     </visual>
+    <collision>
+      <origin xyz="0 0 0" rpy="1.5708 0 0"/>
+      <geometry>
+        <cylinder radius="${wheel_radius}" length="${wheel_width}"/>
+      </geometry>
+    </collision>
+    <inertial>
+      <mass value="0.2"/>
+      <inertia
+        ixx="0.0002" ixy="0.0" ixz="0.0"
+        iyy="0.0002" iyz="0.0"
+        izz="0.0001"/>
+    </inertial>
   </link>
   <!-- left wheel joint -->
@@ -63,5 +112,5 @@
   <link name="right_wheel_link">
     <visual>
-      <origin xyz="0 0 0" rpy="1.5709 0 0"/>
+      <origin xyz="0 0 0" rpy="1.5708 0 0"/>
       <geometry>
         <cylinder radius="${wheel_radius}" length="${wheel_width}"/>
@@ -71,4 +120,17 @@
       </material>
     </visual>
+    <collision>
+      <origin xyz="0 0 0" rpy="1.5708 0 0"/>
+      <geometry>
+        <cylinder radius="${wheel_radius}" length="${wheel_width}"/>
+      </geometry>
+    </collision>
+    <inertial>
+      <mass value="0.2"/>
+        <inertia
+          ixx="0.0002" ixy="0.0" ixz="0.0"
+          iyy="0.0002" iyz="0.0"
+          izz="0.0001"/>
+    </inertial>
   </link>
   <!-- right wheel join -->

Commit message: update before taking Udemy ros2

File: src/my_minimal_robot_description/urdf/minimal_robot.xacro (robot description, xacro)
@@ -45,4 +45,29 @@
     </inertial>
   </link>
+    <!-- ========== LiDAR frame ========== -->
+  <link name="lidar_link">
+    <visual>
+      <origin xyz="0 0 0" rpy="0 0 0"/>
+      <geometry>
+        <cylinder length="0.05" radius="0.035"/>
+      </geometry>
+    </visual>
+    <collision>
+      <origin xyz="0 0 0" rpy="0 0 0"/>
+      <geometry>
+        <cylinder length="0.05" radius="0.035"/>
+      </geometry>
+    </collision>
+    <inertial>
+      <mass value="0.2"/>
+      <origin xyz="0 0 0" rpy="0 0 0"/>
+      <inertia ixx="1e-4" ixy="0" ixz="0" iyy="1e-4" iyz="0" izz="1e-4"/>
+    </inertial>
+  </link>
+  <joint name="lidar_joint" type="fixed">
+    <origin xyz="0.18 0 0.15" rpy="0 0 0"/>
+    <parent link="base_link"/>
+    <child link="lidar_link"/>
+  </joint>
   <!-- sensor_link -->
   <link name="sensor_link">
@@ -141,3 +166,25 @@
     <axis xyz="0 1 0"/>
   </joint>
+  <!-- Gazebo Sim LiDAR -->
+  <gazebo reference="lidar_link">
+    <sensor name="lidar" type="gpu_lidar">
+      <always_on>true</always_on>
+      <update_rate>10</update_rate>
+      <visualize>false</visualize>
+      <topic>/scan</topic>
+      <gpu_lidar>
+        <horizontal>
+          <samples>360</samples>
+          <resolution>1</resolution>
+          <min_angle>-3.14159265</min_angle>
+          <max_angle>3.14159265</max_angle>
+        </horizontal>
+        <range>
+          <min>0.12</min>
+          <max>12.0</max>
+          <resolution>0.01</resolution>
+        </range>
+      </gpu_lidar>
+    </sensor>
+  </gazebo>
 </robot>
