Commit message: update my_robot description and bringup folder

File: src/my_robot_description/urdf/common_properties.xacro (robot description, xacro)
@@ -7,3 +7,30 @@
             <color rgba="0.5 0.5 0.5 1.0"/>
     </material>
+    <xacro:macro name="box_inertia" params="m l w h xyz rpy">
+        <inertial>
+                <origin xyz="${xyz}" rpy="${rpy}" />
+                <mass value="${m}" />
+                <inertia ixx="${(1/12.0)*m*(h*h + w*w)}" ixy="0.0" ixz="0.0"
+                         iyy="${(1/12.0)*m*(h*h + l*l)}" iyz="0.0"
+                         izz="${(1/12.0)*m*(w*w + l*l)}"/>
+        </inertial>
+    </xacro:macro>
+    <xacro:macro name="cylinder_inertia" params="m r h xyz rpy">
+        <inertial>
+                <origin xyz="${xyz}" rpy="${rpy}" />
+                <mass value="${m}" />
+                <inertia ixx="${(1/12.0)*m*(3*r*r + h*h)}" ixy="0.0" ixz="0.0"
+                         iyy="${(1/12.0)*m*(3*r*r + h*h)}" iyz="0.0"
+                         izz="${(1/2.0)*m*r*r}"/>
+        </inertial>
+    </xacro:macro>
+    <xacro:macro name="sphere_inertia" params="m r xyz rpy">
+        <inertial>
+                <origin xyz="${xyz}" rpy="${rpy}" />
+                <mass value="${m}" />
+                <inertia ixx="${(2/5.0)*m*r*r}" ixy="0.0" ixz="0.0"
+                         iyy="${(2/5.0)*m*r*r}" iyz="0.0"
+                         izz="${(2/5.0)*m*r*r}"/>
+        </inertial>
+    </xacro:macro>
 </robot>

File: src/my_robot_description/urdf/mobile_base.xacro (robot description, xacro)
@@ -6,4 +6,5 @@
     <xacro:property name="wheel_radius" value="0.1"/>
     <xacro:property name="wheel_length" value="0.05"/>
+    <!--<xacro:property name="pi" value="3.141592653589793"/>-->
     <link name="base_footprint"/>
     <link name="base_link">
@@ -15,4 +16,11 @@
             <material name="green" />
         </visual>
+        <collision>
+            <geometry>
+                <box size="${base_length} ${base_width} ${base_height}"/>
+            </geometry>
+            <origin xyz="0 0 ${base_height/2}" rpy="0 0 0"/>
+        </collision>
+        <xacro:box_inertia m="5.0" l="${base_length}" w="${base_width}" h="${base_height}" xyz="0 0 ${base_height/2}" rpy ="0 0 0"/>
     </link>
     <xacro:macro name="wheel_link" params="prefix">
@@ -25,4 +33,11 @@
                 <material name="grey" />
             </visual>
+            <collision>
+                <geometry>
+                    <cylinder radius="${wheel_radius}" length="${wheel_length}"/>
+                </geometry>
+                <origin xyz="0.0 0.0 0.0" rpy="${pi/2} 0 0"/>
+            </collision>
+            <xacro:cylinder_inertia m="1.0" r="${wheel_radius}" h="${wheel_length}" xyz="0.0 0.0 0.0" rpy="${pi/2} 0 0"/>
         </link>
     </xacro:macro>
@@ -37,4 +52,11 @@
             <material name="grey" />
         </visual>
+        <collision>
+            <geometry>
+                <sphere radius="${wheel_radius / 2}"/>
+            </geometry>
+            <origin xyz="0.0 0.0 0.0" rpy="0 0 0"/>
+        </collision>
+        <xacro:sphere_inertia m="0.5" r="${wheel_radius / 2}" xyz="0.0 0.0 0.0" rpy="0 0 0"/>
     </link>
     <joint name="base_footprint_to_base_link" type="fixed">

File: src/my_robot_description/urdf/my_robot.urdf.xacro (robot description, xacro)
@@ -3,3 +3,4 @@
     <xacro:include filename="common_properties.xacro"/>
     <xacro:include filename="mobile_base.xacro"/>
+    <xacro:include filename="mobile_base_gazebo.xacro" />
 </robot>

Commit message: added a arm on the robot

File: src/my_robot_description/urdf/common_properties.xacro (robot description, xacro)
@@ -6,4 +6,10 @@
     <material name="grey">
             <color rgba="0.5 0.5 0.5 1.0"/>
+    </material>
+    <material name="yellow">
+            <color rgba="0.8 0.8 0.0 1.0"/>
+    </material>
+    <material name="orange">
+            <color rgba="0.8 0.4 0.0 1.0"/>
     </material>
     <xacro:macro name="box_inertia" params="m l w h xyz rpy">

File: src/my_robot_description/urdf/mobile_base_gazebo.xacro (robot description, xacro)
@@ -23,7 +23,7 @@
             filename="libignition-gazebo-joint-state-publisher-system.so"
             name="ignition::gazebo::systems::JointStatePublisher">
-            <!-- <topic>/joint_states</topic> -->
             <joint_name>base_left_wheel_joint</joint_name>
             <joint_name>base_right_wheel_joint</joint_name>
+            <topic>/joint_states</topic>
         </plugin>
     </gazebo>

File: src/my_robot_description/urdf/my_robot.urdf.xacro (robot description, xacro)
@@ -5,3 +5,4 @@
     <xacro:include filename="mobile_base_gazebo.xacro" />
     <xacro:include filename="camera.xacro" />
+    <xacro:include filename="arm.xacro"/>
 </robot>
